File: KiCAD project 1.0/frogger.sch (KiCad schematic (older format))
At the start: 61 parts, among them J1 USB_B_Micro, J2 USB_B_Mini, J3 Conn_01x02, J4 Conn_01x02, Q1 BC557, Q2 PN2222A, SW1 SW_Push, SW2 SW_Push

Commit message: KiCAD project 1.0
Parts:
- D1, D2, D3: value 1N4007 -> 1N4001
- R10: value 300k -> 100k
- R11: value 100k -> 300k
Changed lines of the file:
@@
 P 3450 3050
 F 0 "D1" H 3450 3267 50  0000 C CNN
-F 1 "1N4007" H 3450 3176 50  0000 C CNN
+F 1 "1N4001" H 3450 3176 50  0000 C CNN
 F 2 "Diode_THT:D_DO-41_SOD81_P10.16mm_Horizontal" H 3450 2875 50  0001 C CNN
 F 3 "http://www.vishay.com/docs/88503/1n4001.pdf" H 3450 3050 50  0001 C CNN
@@
 P 2650 800
 F 0 "D2" H 2650 1017 50  0000 C CNN
-F 1 "1N4007" H 2650 926 50  0000 C CNN
+F 1 "1N4001" H 2650 926 50  0000 C CNN
 F 2 "Diode_THT:D_DO-41_SOD81_P10.16mm_Horizontal" H 2650 625 50  0001 C CNN
 F 3 "http://www.vishay.com/docs/88503/1n4001.pdf" H 2650 800 50  0001 C CNN
@@
 P 2650 1150
 F 0 "D3" H 2650 1367 50  0000 C CNN
-F 1 "1N4007" H 2650 1276 50  0000 C CNN
+F 1 "1N4001" H 2650 1276 50  0000 C CNN
 F 2 "Diode_THT:D_DO-41_SOD81_P10.16mm_Horizontal" H 2650 975 50  0001 C CNN
 F 3 "http://www.vishay.com/docs/88503/1n4001.pdf" H 2650 1150 50  0001 C CNN
@@
 P 4750 1300
 F 0 "R10" H 4818 1346 50  0000 L CNN
-F 1 "300k" H 4818 1255 50  0000 L CNN
+F 1 "100k" H 4818 1255 50  0000 L CNN
 F 2 "Resistor_THT:R_Axial_DIN0207_L6.3mm_D2.5mm_P10.16mm_Horizontal" V 4790 1290 50  0001 C CNN
 F 3 "~" H 4750 1300 50  0001 C CNN
@@
 P 4750 1800
 F 0 "R11" H 4818 1846 50  0000 L CNN
-F 1 "100k" H 4818 1755 50  0000 L CNN
+F 1 "300k" H 4818 1755 50  0000 L CNN
 F 2 "Resistor_THT:R_Axial_DIN0207_L6.3mm_D2.5mm_P10.16mm_Horizontal" V 4790 1790 50  0001 C CNN
 F 3 "~" H 4750 1800 50  0001 C CNN
